Commit message: slam_ran

File: install/car/share/car/description/new_robot.xacro (robot description, xacro)
@@ -17,26 +17,33 @@
     <link name="base_link">
     </link>
+    <joint name = "base_footprint_joint" type="fixed">
+        <parent link = "base_link"/>
+        <child link = "base_footprint"/>
+        <origin xyz = "0 0 0" rpy ="0 0 0"/>
+    </joint>
+    <link name = "base_footprint">
+    </link>
     <!-- CHASSIS LINK -->
     <joint name="chassis_joint" type="fixed">
         <parent link="base_link"/>
         <child link="chassis"/>
-        <origin xyz="-0.1 0 0"/>
+        <origin xyz="-0.15 0 0"/>
     </joint>
     <link name="chassis">
         <visual>
-            <origin xyz="0.15 0 0.075"/>
-            <geometry>
-                <box size="0.3 0.3 0.15"/>
+            <origin xyz="0.2 0 0.1"/>
+            <geometry>
+                <box size="0.4 0.4 0.2"/>
             </geometry>
             <material name="white"/>
         </visual>
         <collision>
-            <origin xyz="0.15 0 0.075"/>
-            <geometry>
-                <box size="0.3 0.3 0.15"/>
-            </geometry>
-        </collision>
-        <xacro:inertial_box mass="0.5" x="0.3" y="0.3" z="0.15">
-            <origin xyz="0.15 0 0.075" rpy="0 0 0"/>
+            <origin xyz="0.2 0 0.1"/>
+            <geometry>
+                <box size="0.4 0.4 0.2"/>
+            </geometry>
+        </collision>
+        <xacro:inertial_box mass="0.8" x="0.4" y="0.4" z="0.2">
+            <origin xyz="0.2 0 0.1" rpy="0 0 0"/>
         </xacro:inertial_box>
     </link>
@@ -45,5 +52,5 @@
         <parent link="chassis"/>
         <child link="camera_box"/>
-        <origin xyz="0.15 0 0.225"/>
+        <origin xyz="0.2 0 0.3"/>
     </joint>
     <link name="camera_box">
@@ -51,5 +58,5 @@
             <origin xyz="0 0 0.05"/>
             <geometry>
-                <box size="0.1 0.1 0.1"/>
+                <box size="0.12 0.12 0.12"/>
             </geometry>
             <material name="orange"/>
@@ -58,8 +65,8 @@
             <origin xyz="0 0 0.05"/>
             <geometry>
-                <box size="0.1 0.1 0.1"/>
-            </geometry>
-        </collision>
-        <xacro:inertial_box mass="0.1" x="0.1" y="0.1" z="0.1">
+                <box size="0.12 0.12 0.12"/>
+            </geometry>
+        </collision>
+        <xacro:inertial_box mass="0.1" x="0.12" y="0.12" z="0.12">
             <origin xyz="0 0 0.05" rpy="0 0 0"/>
         </xacro:inertial_box>
@@ -69,5 +76,5 @@
         <parent link="camera_box"/>
         <child link="camera_link"/>
-        <origin xyz="0 0 0.1"/>
+        <origin xyz="0 0 0.15"/>
     </joint>
     <link name="camera_link">
@@ -104,9 +111,60 @@
         </sensor>
     </gazebo>
+    <!-- LIDAR LINK -->
+    <joint name="lidar_joint" type="fixed">
+        <parent link="chassis"/>
+        <child link="lidar_link"/>
+        <origin xyz="0.2 0 0.2"/>
+    </joint>
+    <link name="lidar_link">
+        <visual>
+            <geometry>
+                <cylinder radius="0.04" length="0.05"/>
+            </geometry>
+            <material name="black"/>
+        </visual>
+        <collision>
+            <geometry>
+                <cylinder radius="0.04" length="0.05"/>
+            </geometry>
+        </collision>
+        <xacro:inertial_cylinder mass="0.1" length="0.05" radius="0.04">
+            <origin xyz="0 0 0" rpy="0 0 0"/>
+        </xacro:inertial_cylinder>
+    </link>
+    <gazebo reference="lidar_link">
+        <sensor name="lidar" type="ray">
+            <pose>0 0 0 0 0 0</pose>
+            <visualize>true</visualize>
+            <update_rate>10</update_rate>
+            <ray>
+                <scan>
+                    <horizontal>
+                        <samples>360</samples>
+                        <resolution>1</resolution>
+                        <min_angle>-3.14159</min_angle>
+                        <max_angle>3.14159</max_angle>
+                    </horizontal>
+                </scan>
+                <range>
+                    <min>0.3</min>
+                    <max>12.0</max>
+                    <resolution>0.01</resolution>
+                </range>
+            </ray>
+            <plugin name="laser_controller" filename="libgazebo_ros_ray_sensor.so">
+                <ros>
+                    <argument>~/out:=scan</argument>
+                </ros>
+                <output_type>sensor_msgs/LaserScan</output_type>
+                <frame_name>lidar_link</frame_name>
+            </plugin>
+        </sensor>
+    </gazebo>
     <!-- LEFT WHEEL LINK -->
     <joint name="left_wheel_joint" type="continuous">
         <parent link="base_link"/>
         <child link="left_wheel"/>
-        <origin xyz="0 0.175 0" rpy="-${pi/2} 0 0" />
+        <origin xyz="0 0.225 0" rpy="-${pi/2} 0 0" />
         <axis xyz="0 0 1"/>
     </joint>
@@ -114,5 +172,5 @@
         <visual>
             <geometry>
-                <cylinder radius="0.05" length="0.04"/>
+                <cylinder radius="0.065" length="0.05"/>
             </geometry>
             <material name="blue"/>
@@ -120,8 +178,8 @@
         <collision>
             <geometry>
-                <cylinder radius="0.05" length="0.04"/>
-            </geometry>
-        </collision>
-        <xacro:inertial_cylinder mass="0.1" length="0.04" radius="0.05">
+                <cylinder radius="0.065" length="0.05"/>
+            </geometry>
+        </collision>
+        <xacro:inertial_cylinder mass="0.1" length="0.05" radius="0.065">
             <origin xyz="0 0 0" rpy="0 0 0"/>
         </xacro:inertial_cylinder>
@@ -134,5 +192,5 @@
         <parent link="base_link"/>
         <child link="right_wheel"/>
-        <origin xyz="0 -0.175 0" rpy="-${pi/2} 0 0" />
+        <origin xyz="0 -0.225 0" rpy="-${pi/2} 0 0" />
         <axis xyz="0 0 1"/>
     </joint>
@@ -140,5 +198,5 @@
         <visual>
             <geometry>
-                <cylinder radius="0.05" length="0.04"/>
+                <cylinder radius="0.065" length="0.05"/>
             </geometry>
             <material name="blue"/>
@@ -146,8 +204,8 @@
         <collision>
             <geometry>
-                <cylinder radius="0.05" length="0.04"/>
-            </geometry>
-        </collision>
-        <xacro:inertial_cylinder mass="0.1" length="0.04" radius="0.05">
+                <cylinder radius="0.065" length="0.05"/>
+            </geometry>
+        </collision>
+        <xacro:inertial_cylinder mass="0.1" length="0.05" radius="0.065">
             <origin xyz="0 0 0" rpy="0 0 0"/>
         </xacro:inertial_cylinder>
@@ -160,10 +218,10 @@
         <parent link="chassis"/>
         <child link="caster_wheel"/>
-        <origin xyz="0.24 0 0"/>
+        <origin xyz="0.32 0 0"/>
     </joint>
     <link name="caster_wheel">
         <visual>
             <geometry>
-                <sphere radius="0.05"/>
+                <sphere radius="0.065"/>
             </geometry>
             <material name="black"/>
@@ -171,8 +229,8 @@
         <collision>
             <geometry>
-                <sphere radius="0.05"/>
-            </geometry>
-        </collision>
-        <xacro:inertial_sphere mass="0.1" radius="0.05">
+                <sphere radius="0.065"/>
+            </geometry>
+        </collision>
+        <xacro:inertial_sphere mass="0.1" radius="0.065">
             <origin xyz="0 0 0" rpy="0 0 0"/>
         </xacro:inertial_sphere>
